Commit message: Added spherical proxy balls and PSMs tip for collision checking

File: dvrk_model/model/psm.urdf.xacro (robot description, xacro)
@@ -250,4 +250,9 @@
         </geometry>
       </visual>
+     <collision>
+       <geometry>
+         <mesh filename="package://dvrk_model/meshes/psm/sphere_20mm.dae"/>
+       </geometry>
+     </collision>
     </link>
   </xacro:macro>

Commit message: Added more SPRs for different diameters

File: dvrk_model/model/psm.urdf.xacro (robot description, xacro)
@@ -247,12 +247,13 @@
         <origin rpy="0 3.1516 0" xyz="0 0 0"/>
         <geometry>
-          <mesh filename="package://dvrk_model/meshes/psm/tool_wrist_sca_link_2.dae"/>
-        </geometry>
-      </visual>
-     <collision>
+          <mesh filename="package://dvrk_model/meshes/psm/sphere_50mm.dae"/>
+          <!--mesh filename="package://dvrk_model/meshes/psm/tool_wrist_sca_link_2.dae"/-->
+        </geometry>
+      </visual>
+     <!--collision>
        <geometry>
-         <mesh filename="package://dvrk_model/meshes/psm/sphere_20mm.dae"/>
+         <mesh filename="package://dvrk_model/meshes/psm/sphere_50mm.dae"/>
        </geometry>
-     </collision>
+     </collision-->
     </link>
   </xacro:macro>

Commit message: Added meshs for tip collision detection

File: dvrk_model/model/psm.urdf.xacro (robot description, xacro)
@@ -229,4 +229,5 @@
         <origin rpy="0 0 0" xyz="0 0 0"/>
         <geometry>
+          <!--mesh filename="package://dvrk_model/meshes/psm/needle.dae"/-->
           <mesh filename="package://dvrk_model/meshes/psm/tool_wrist_sca_link_2.dae"/>
         </geometry>
@@ -247,4 +248,5 @@
         <origin rpy="0 3.1516 0" xyz="0 0 0"/>
         <geometry>
+	  <!--mesh filename="package://dvrk_model/meshes/psm/needle.stl"/-->
           <mesh filename="package://dvrk_model/meshes/psm/sphere_50mm.dae"/>
           <!--mesh filename="package://dvrk_model/meshes/psm/tool_wrist_sca_link_2.dae"/-->
@@ -253,5 +255,5 @@
      <!--collision>
        <geometry>
-         <mesh filename="package://dvrk_model/meshes/psm/sphere_50mm.dae"/>
+         <mesh filename="package://dvrk_model/meshes/psm/needle.dae"/>
        </geometry>
      </collision-->
